File: eagle/SensorBoard/airball_sensor_board_v3.brd (EAGLE design)
At the start: 139.7 x 38.1 mm, 28 parts

Commit message: Cleanup of EAGLE libraries
Several parts were added to the unrelated library microbuilder.lbr;
migrate those to a new airball.lbr library file, and delete
microbuilder. Adjust airball_sensor_board_v3 to reference the new
library and adjust schematic device placement for minor cleanups.
Parts:
- BARO, DP0, DPA, DPB: device microbuilder:ALL_SENSORS_E1BD_8PIN_THRU -> airball:ALL_SENSORS_E1BD_8PIN_THRU
- JP1: device jcole:USB_MICRO_B_TYCO -> airball:USB_MICRO_B_TYCO
- U$2: device microbuilder:SPARKFUN_FIO_V3 -> airball:SPARKFUN_FIO_V3
- U1: device microbuilder:TSSOP24 -> airball:TSSOP24
Changed lines of the file:
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@@
 <?xml version="1.0" encoding="utf-8"?>
 <!DOCTYPE eagle SYSTEM "eagle.dtd">
-<eagle version="8.5.2">
+<eagle version="8.6.0">
 <drawing>
 <settings>
-<setting alwaysvectorfont="no"/>
+<setting alwaysvectorfont="yes"/>
 <setting keepoldvectorfont="yes"/>
 <setting verticaltext="up"/>
@@
 <layer number="59" name="tCarbon" color="7" fill="1" visible="no" active="no"/>
 <layer number="60" name="bCarbon" color="7" fill="1" visible="no" active="no"/>
+<layer number="88" name="SimResults" color="9" fill="1" visible="no" active="no"/>
+<layer number="89" name="SimProbes" color="9" fill="1" visible="no" active="no"/>
 <layer number="90" name="Modules" color="5" fill="1" visible="no" active="no"/>
 <layer number="91" name="Nets" color="2" fill="1" visible="no" active="no"/>
@@
 </autorouter>
 <elements>
-<element name="BARO" library="microbuilder" package="ALL_SENSORS_E1BD_8PIN_THRU" value="" x="72.39" y="22.86"/>
-<element name="DPA" library="microbuilder" package="ALL_SENSORS_E1BD_8PIN_THRU" value="" x="50.165" y="22.86"/>
-<element name="DPB" library="microbuilder" package="ALL_SENSORS_E1BD_8PIN_THRU" value="" x="27.94" y="22.86"/>
+<element name="BARO" library="airball" package="ALL_SENSORS_E1BD_8PIN_THRU" value="" x="72.39" y="22.86"/>
+<element name="DPA" library="airball" package="ALL_SENSORS_E1BD_8PIN_THRU" value="" x="50.165" y="22.86"/>
+<element name="DPB" library="airball" package="ALL_SENSORS_E1BD_8PIN_THRU" value="" x="27.94" y="22.86"/>
 <element name="C2" library="SparkFun-Capacitors" package="0603" value="0.1uF" x="61.2775" y="24.13" smashed="yes" rot="R180">
 <attribute name="NAME" x="61.2775" y="23.368" size="0.6096" layer="25" font="vector" ratio="20" rot="R180" align="bottom-center"/>
@@
 <attribute name="PROD_ID" value="RES-07857" x="16.8275" y="19.05" size="1.778" layer="27" rot="R180" display="off"/>
 </element>
-<element name="DP0" library="microbuilder" package="ALL_SENSORS_E1BD_8PIN_THRU" value="" x="94.615" y="22.86"/>
+<element name="DP0" library="airball" package="ALL_SENSORS_E1BD_8PIN_THRU" value="" x="94.615" y="22.86"/>
 <element name="C1" library="SparkFun-Capacitors" package="0603" value="0.1uF" x="83.5025" y="24.13" smashed="yes" rot="R180">
 <attribute name="NAME" x="83.5025" y="23.368" size="0.6096" layer="25" font="vector" ratio="20" rot="R180" align="bottom-center"/>
@@
 <attribute name="PROD_ID" value="RES-07857" x="83.5025" y="19.05" size="1.778" layer="27" rot="R180" display="off"/>
 </element>
-<element name="U$2" library="microbuilder" package="SPARKFUN_FIO_V3" value="SPARKFUN_FIO_V3" x="78.74" y="19.05" smashed="yes" rot="MR90"/>
-<element name="U1" library="microbuilder" package="TSSOP24" value="" x="114.3" y="20.32" smashed="yes" rot="R270">
+<element name="U$2" library="airball" package="SPARKFUN_FIO_V3" value="SPARKFUN_FIO_V3" x="78.74" y="19.05" smashed="yes" rot="MR90"/>
+<element name="U1" library="airball" package="TSSOP24" value="" x="114.3" y="20.32" smashed="yes" rot="R270">
 <attribute name="VALUE" x="112.2172" y="15.1338" size="1.016" layer="27" ratio="10"/>
 </element>
@@
 <attribute name="PROD_ID" value="RES-07857" x="121.285" y="22.5425" size="1.778" layer="27" display="off"/>
 </element>
-<element name="JP1" library="jcole" package="USB_MICRO_B_TYCO" value="USB_MICROB_PLUG" x="138.1125" y="26.035" smashed="yes" rot="R90"/>
+<element name="JP1" library="airball" package="USB_MICRO_B_TYCO" value="USB_MICROB_PLUG" x="138.1125" y="26.035" smashed="yes" rot="R90"/>
 </elements>
 <signals>
