File: eagle/DisplayBoard/airball_display_board_v1.sch (EAGLE design)
At the start: 10 parts, among them J1 MICRO-SD_CARD_SOCKET, J2 USB_A_SMT_FEMALE_NS

Commit message: Another WIP commit for display v1
Parts:
- removed U$1: RPI_CM3-TYCO1376408, airball:RPI_CM3-TYCO1376408
- removed U$2: TFP401, airball:TFP401
- removed U$3: TFT_40PIN_FFC, airball:TFT_40PIN_FFC
- removed U$5: TI_TPS61169, airball:TI_TPS61169
- removed U$6: PAM2306, airball:PAM2306
- added C1, C2, C3, C4, C6: 10uF, SparkFun-Capacitors:10UF-POLAR-EIA3216-16V-10%(TANT)
- added C5: 0.1uF, SparkFun-Capacitors:0.1UF-0603-25V-5%
- added D1: NSR0240H, airball:DIODE-SCHOTTKY-SOD323
- added J3: AVR_SPI_PROG_3X2PTH, SparkFun-Connectors:AVR_SPI_PROG_3X2PTH
- added L1, L2, L3: 4.7uH, airball:INDUCTOR-SMD_4X4
- added Q1, Q2: DMG1012T, airball:DMG1012T
- added R1, R10, R2, R3, R4, R5, R8, R9: 100k, SparkFun-Resistors:100KOHM-0603-1/10W-1%
- added R11, R12, R6, R7: 4.7k, SparkFun-Resistors:4.7KOHM-0603-1/10W-1%
- added R13: 5R1, SparkFun-Resistors:RESISTOR0603
- added R14: 10k, SparkFun-Resistors:10KOHM-0603-1/10W-1%
- added S1: (no value), SparkFun-Switches:SWITCH-SPDT-SMD-RIGHT-ANGLE
- added U1: RPI_CM3-TYCO1376408, airball:RPI_CM3-TYCO1376408
- added U2: TFP401A, airball:TFP401-POWER_LITE
- added U3: TFT_40PIN_FFC-TOP, airball:TFT_40PIN_FFC-TOP
- added U4: ATtiny85, airball:ATTINY25/45/85
- added U5: TPS61169, airball:TPS61169
- added U6: PAM2306AYPKE, airball:PAM2306
- added U7: LM3880MF-1AB, airball:LM3880
- added U8: 24LC02B, airball:24LC02B
- added U9: FSUSB42, airball:FSUSB42
- J1: value MICRO-SD_CARD_SOCKET -> (none); device SparkFun-Connectors:MICRO-SD_CARD_SOCKET -> airball:MICRO-SD-SD4
Connections:
- removed net N$27: U$2EVEN.QG7, U$3.G7
- removed net N$28: U$2EVEN.QB0, U$3.B0
- removed net N$29: U$2EVEN.QB1, U$3.B1
- removed net N$30: U$2EVEN.QB2, U$3.B2
- removed net N$31: U$2EVEN.QB3, U$3.B3
- removed net N$32: U$2EVEN.QB4, U$3.B4
- removed net N$33: U$2EVEN.QB5, U$3.B5
- removed net N$34: U$2EVEN.QB6, U$3.B6
- removed net N$35: U$2EVEN.QB7, U$3.B7
- removed net N$36: U$2CONTROL.DE, U$3.DE
- removed net N$37: U$2CONTROL.ODCK, U$3.PCLK
- removed net N$38: U$2CONTROL.HSYNC, U$3.HSYNC
- removed net N$39: U$2CONTROL.VSYNC, U$3.VSYNC
- removed net N$40: U$2CONTROL.SCDT, U$3.ENABLE
- new net B0: U2EVEN.QB0, U3.B0
- new net B1: U2EVEN.QB1, U3.B1
- new net B2: U2EVEN.QB2, U3.B2
- new net B3: U2EVEN.QB3, U3.B3
- new net B4: U2EVEN.QB4, U3.B4
- new net B5: U2EVEN.QB5, U3.B5
- new net B6: U2EVEN.QB6, U3.B6
- new net B7: U2EVEN.QB7, U3.B7
- new net BKL_LED_A: C6.+, D1.C, U3.LED_A
- new net BKL_LED_K: R13.2, U3.LED_K, U5.FB
- new net BKL_MISO: J3.1, U4.PB1
- new net BKL_MOSI: J3.4, R7.2, U4.PB0
- new net BKL_RST: J3.5, U4.!RST
- new net BKL_SCK: J3.3, R6.2, U4.PB2
- new net DE: U2CONTROL.DE, U3.DE
- new net EMMC_DISABLE: Q1.D, U1CM3.!EMMC_DISABLE
- new net EMMC_EN: Q2.G, R5.1, U1CM3.!EMMC_EN
- new net EN_1V8: R2.1, U6CH2.EN, U7.FLAG2
- new net EN_3V3: R1.1, U6CH1.EN, U7.FLAG1
- new net G0: U2EVEN.QG0, U3.G0
- new net G1: U2EVEN.QG1, U3.G1
- new net G2: U2EVEN.QG2, U3.G2
- new net G3: U2EVEN.QG3, U3.G3
- new net G4: U2EVEN.QG4, U3.G4
- new net G5: U2EVEN.QG5, U3.G5
- new net G6: U2EVEN.QG6, U3.G6
- new net G7: U2EVEN.QG7, U3.G7
- new net GND: C1.-, C2.-, C3.-, C4.-, C5.2, C6.-, J1.GND, J2.GND, J2.SHIELD, J3.6, JP1.GND, Q2.S, R10.1, R13.1, R3.1, R4.1, R8.1, R9.1, S1.S, U1CM3.GND, U1CM3.OTGID, U2CORE.AGND, U2CORE.DFO, U2CORE.DGND, U2CORE.OCK_INV, U2CORE.OGND, U2CORE.PGND, U2CORE.PIXS, U2CORE.THERMAL, U3.GND, U4.GND, U5.GND, U6CH1.GND, U6CH2.GND, U7.GND, U8.GND, U8.WP, U9.!OE, U9.GND, XB1.GND
- new net HDMI_EDID_SCL: U1HDMI.SCL, U8.SCL
- new net HDMI_EDID_SDA: U1HDMI.SDA, U8.SDA
- new net HSYNC: U2CONTROL.HSYNC, U3.HSYNC
- new net LED_ACT: Q1.S, Q2.D
- new net PCLK: U2CONTROL.ODCK, U3.PCLK
- new net R0: U2EVEN.QR0, U3.R0
- new net R1: U2EVEN.QR1, U3.R1
- new net R2: U2EVEN.QR2, U3.R2
- new net R3: U2EVEN.QR3, U3.R3
- new net R4: U2EVEN.QR4, U3.R4
- new net R5: U2EVEN.QR5, U3.R5
- new net R6: U2EVEN.QR6, U3.R6
- new net R7: U2EVEN.QR7, U3.R7
- new net RXD0: U1CM3.GPIO15, XB1.DOUT
- new net SCDT: U2CONTROL.SCDT, U3.ENABLE
- new net SCL1: R12.2, R6.1, U1CM3.GPIO3
- new net SDA1: R11.2, R7.1, U1CM3.GPIO2
- new net TXD0: U1CM3.GPIO14, XB1.DIN/!CONFIG
- new net USB_A_N: J2.D-, U9.D1-
- new net USB_A_P: J2.D+, U9.D1+
- new net USB_BOOT_EN: Q1.G, R4.2
- new net USB_B_N: JP1.D-, U9.D2-
- new net USB_B_P: JP1.D+, U9.D2+
- new net USB_N: U1CM3.D-, U9.D-
- new net USB_P: U1CM3.D+, U9.D+
- new net VCC_1V8: C2.+, L2.2, R5.2, U1CM3.VCC_1V8, U6CH2.FB
- new net VCC_3V3: C1.+, J1.VCC, L1.2, R11.1, R12.1, R14.1, U1CM3.VCC_3V3, U1CM3.VDAC, U1CM3.VDD_GPIO0_27, U1CM3.VDD_GPIO28_45, U1CM3.VDD_SDX, U2CORE.!STAG, U2CORE.AVDD, U2CORE.DVDD, U2CORE.OVDD, U2CORE.PVDD, U2CORE.RSVD, U2CORE.ST, U3.VDD, U6CH1.FB, U8.VCC, U9.VCC, XB1.VCC
- new net VCC_5V0: C3.+, C4.+, J2.VBUS, J3.2, JP1.VCC, L3.1, R1.2, R2.2, U1CM3.VBAT, U4.VCC, U5.VIN, U6CH1.VIN, U6CH2.VIN, U7.VCC
- new net VSYNC: U2CONTROL.VSYNC, U3.VSYNC
- net N$1: now also J1.CLK, U1SDX.CLK; no longer J1.SCK, U$1SDX.CLK
- net N$10: now also U1HDMI.CLK+, U2INPUT.CLK+; no longer U$1HDMI.CLK_P, U$2INPUT.C_P
- net N$11: now also U1HDMI.CLK-, U2INPUT.CLK-; no longer U$1HDMI.CLK_N, U$2INPUT.C_N
- net N$12: now also J1.D1, U1SDX.D1; no longer U$2EVEN.QR0, U$3.R0
- net N$13: now also J1.D2, U1SDX.D2; no longer U$2EVEN.QR1, U$3.R1
- net N$14: now also J1.D3, U1SDX.D3; no longer U$2EVEN.QR2, U$3.R2
- net N$15: now also L1.1, U6CH1.LX; no longer U$2EVEN.QR3, U$3.R3
- net N$16: now also L2.1, U6CH2.LX; no longer U$2EVEN.QR4, U$3.R4
- net N$17: now also C5.1, U7.EN; no longer U$2EVEN.QR5, U$3.R5
- net N$18: now also R3.2, U1CM3.GPIO29; no longer U$2EVEN.QR6, U$3.R6
- net N$19: now also XB1.ON/!SLEEP; no longer U$2EVEN.QR7, U$3.R7
- net N$2: now also J1.CMD, U1SDX.CMD; no longer J1.DI, U$1SDX.D0
- net N$20: now also XB1.ASSOC/AD5/DIO5; no longer U$2EVEN.QG0, U$3.G0
- net N$21: now also R8.2, U1CM3.GPIO28; no longer U$2EVEN.QG1, U$3.G1
- net N$22: now also U4.PB4, U5.CTRL; no longer U$2EVEN.QG2, U$3.G2
- net N$23: now also R9.2, U1CM3.GPIO45; no longer U$2EVEN.QG3, U$3.G3
- net N$24: now also R10.2, U1CM3.GPIO44; no longer U$2EVEN.QG4, U$3.G4
- net N$25: now also D1.A, L3.2, U5.SW; no longer U$2EVEN.QG5, U$3.G5
- net N$26: now also R14.2, S1.P, U9.SEL; no longer U$2EVEN.QG6, U$3.G6
- net N$3: now also J1.D0, U1SDX.D0; no longer J1.DO, U$1SDX.D1
- net N$4: now also U1HDMI.D2+, U2INPUT.D2+; no longer U$1HDMI.D2_P, U$2INPUT.D2_P
- net N$5: now also U1HDMI.D2-, U2INPUT.D2-; no longer U$1HDMI.D2_N, U$2INPUT.D2_N
- net N$6: now also U1HDMI.D1+, U2INPUT.D1+; no longer U$1HDMI.D1_P, U$2INPUT.D1_P
- net N$7: now also U1HDMI.D1-, U2INPUT.D1-; no longer U$1HDMI.D1_N, U$2INPUT.D1_N
- net N$8: now also U1HDMI.D0+, U2INPUT.D0+; no longer U$1HDMI.D0_P, U$2INPUT.D0_P
- net N$9: now also U1HDMI.D0-, U2INPUT.D0-; no longer U$1HDMI.D0_N, U$2INPUT.D0_N
Other:
- note added: "Display"
- note added: "HDMI EDID EEPROM (optional)"
- note added: "HDMI Input from CM3"
- note added: "HDMI to PanelBus Convertor"
- note added: "Input"
- note added: "I²C Input from Raspberry Pi"
- note added: "I²C LED Backlight Control for TFT"
- note added: "Main Power Supply/Regulation"
- note added: "Output"
- note added: "PWM Output to backlight (~25.6V)"
- note added: "PanelBus Output to TFT"
- note added: "Power Regulation"
- note added: "Processing/Radio"
- note added: "Raspberry Pi 3 pin mappings: * GPIO2 = SDA1 * GPIO3 = SCL1 * GPIO14 = TXD0 * GPIO15 = RXD0"
- note added: "Raspberry Pi Compute Module"
- note added: "Startup Sequencing"
- note added: "TODO: * Add decoupling"
- note added: "TODO: * Add decoupling * USB connections * Power status LEDs * XBee status LEDs * Add UI switches etc."
- note added: "Touch Screen not supported"
- note added: "USB A/µB Ports and Selector"
- note added: "USB/eMMC Boot Selection"
- note added: "Voltage Regulation"
- note added: "XBee Radio"
- note added: "µSD Storage (optional)"
- note added: "×"
- note removed: "LED Backlight Supply"

Commit message: Airball Display Board v1 as built
Parts:
- removed J2: USB_A_SMT_FEMALE_NS, SparkFun-Connectors:USB_A_SMT_FEMALE_NS
- removed JP1: USB_MICROB_PLUG, airball:USB_MICROB_PLUG
- added BT1: (no value), SparkFun-Batteries:BATTERY-12MM_SMD
- added C10, C11, C12, C13, C14, C15, C16, C17, C21, C22, C7, C8, C9: 0.1uF, SparkFun-Capacitors:0.1UF-0603-25V-5%
- added C18, C19, C20: 47uF, SparkFun-Capacitors:47UF-POLAR-EIA3528-10V-10%
- added D2, D3, D4, D5, D6: (no value), SparkFun-LED:LED0603
- added R15, R21, R22: 4.7k, SparkFun-Resistors:4.7KOHM-0603-1/10W-1%
- added R16, R17, R18, R19, R20: 330, SparkFun-Resistors:330OHM-0603-1/10W-1%
- added S2: (no value), SparkFun-Switches:SWITCH-SPDT-SMD-RIGHT-ANGLE
- added TP_1V8, TP_3V3, TP_5V0, TP_BKL_LED_A, TP_BKL_LED_K, TP_GND: TEST-POINT3X5, SparkFun-Connectors:TEST-POINT3X5
- added U$1: (no value), airball:ENCODER_WITH_SWITCH
- added U10: DS3231, airball:DS3231
- added U11, U12: (no value), airball:LTC4411
- added USB_A: USB_A, airball:USB_A
- added USB_B_1, USB_B_2: USB_MICROB_PLUG, airball:USB_MICROB_PLUG
- added VR1: 10k, airball:POTENTIOMETERPTV09A
- J1: device airball:MICRO-SD-SD4 -> airball:MICRO-SD-SD4-MOLEX_104031
- U1: value RPI_CM3-TYCO1376408 -> RPI_CM3-AMP_1473149; device airball:RPI_CM3-TYCO1376408 -> airball:RPI_CM3-AMP_1473149
- U3: value TFT_40PIN_FFC-TOP -> TFT_40PIN_FFC-BOT; device airball:TFT_40PIN_FFC-TOP -> airball:TFT_40PIN_FFC-BOT
- XB1: value XBEE-PRO-SMD -> XBEE-PRO; device airball:XBEE-PRO-SMD -> airball:XBEE-PRO
Connections:
- net N$1 renamed SD_CLK
- net N$10 renamed HDMI_CLK_P
- net N$11 renamed HDMI_CLK_N
- net N$12 renamed SD_D1
- net N$13 renamed SD_D2
- net N$14 renamed SD_D3
- net N$15 renamed L_VCC_3V3
- net N$16 renamed L_VCC_1V8
- net N$18 renamed PD_GPIO29
- net N$2 renamed SD_CMD
- net N$21 renamed PD_GPIO28
- net N$22 renamed BKL_PWM
- net N$23 renamed PD_GPIO45
- net N$24 renamed PD_GPIO44
- net N$25 renamed L_BKL
- net N$3 renamed SD_D0
- net N$4 renamed HDMI_D2_P
- net N$5 renamed HDMI_D2_N
- net N$6 renamed HDMI_D1_P
- net N$7 renamed HDMI_D1_N
- net N$8 renamed HDMI_D0_P
- net N$9 renamed HDMI_D0_N
- removed net N$19: XB1.ON/!SLEEP
- removed net N$20: XB1.ASSOC/AD5/DIO5
- new net BKL_ADJ: U4.PB3, VR1.S
- new net ENC_A: R7.2, U$1.A, U1CM3.GPIO20
- new net ENC_B: R15.2, U$1.B, U1CM3.GPIO21
- new net ENC_SW: R6.2, U$1.SW+, U1CM3.GPIO22
- new net RTC_VBAT: BT1.+, U10.VBAT
- new net R_POWER: D5.A, R19.1
- new net R_SD_ACT: D6.A, R20.1
- new net R_XBEE_ASSOC: D2.A, R16.1
- new net R_XBEE_ON: D4.A, R18.1
- new net R_XBEE_RSSI: D3.A, R17.1
- new net USB_A_VCC: U12.IN, USB_B_1.VCC
- new net USB_B_VCC: U11.IN, USB_B_2.VCC
- new net XBEE_ASSOC: R16.2, XB1.ASSOC/AD5/DIO5
- new net XBEE_ON: R18.2, XB1.ON/!SLEEP
- new net XBEE_RSSI: R17.2, XB1.PWM0/RSSI
- new net XBEE_SLEEP_RQ: U1CM3.GPIO23, XB1.!DTR!/SLEEP_RQ/DI8
- net BKL_LED_A: now also TP_BKL_LED_A.1
- net BKL_LED_K: now also TP_BKL_LED_K.1
- net BKL_MOSI: no longer R7.2
- net BKL_SCK: no longer R6.2
- net GND: now also BT1.-, C10.1, C11.2, C12.2, C13.2, C14.2, C15.2, C16.2, C17.2, C18.-, C19.-, C20.-, C21.2, C22.2, C7.2, C8.2, C9.2, D2.C, D3.C, D4.C, D5.C, J1.CD1, J1.CD2, R6.1, S1.P, TP_GND.1, U$1.C, U10.GND, U11.CTL, U11.GND, U12.CTL, U12.GND, USB_A.GND, USB_B_1.GND, USB_B_2.GND, VR1.A; no longer J2.GND, J2.SHIELD, JP1.GND, S1.S
- net HDMI_EDID_SCL: now also R22.1
- net HDMI_EDID_SDA: now also R21.1
- net LED_ACT: now also D6.C
- net N$26: now also S1.O; no longer S1.P
- net SCL1: now also U10.SCL; no longer R6.1
- net SDA1: now also U10.SDA; no longer R7.1
- net USB_A_N: now also USB_A.D-; no longer J2.D-
- net USB_A_P: now also USB_A.D+; no longer J2.D+
- net USB_BOOT_EN: now also S2.O
- net USB_B_N: now also USB_B_1.D-; no longer JP1.D-
- net USB_B_P: now also USB_B_1.D+; no longer JP1.D+
- net VCC_1V8: now also C11.1, S2.P, TP_1V8.1
- net VCC_3V3: now also C10.2, C12.1, C15.1, C16.1, C17.1, C18.+, C19.+, C20.+, C21.1, C22.1, C9.1, R15.1, R20.2, R7.1, TP_3V3.1, U$1.SW-, U10.VCC; no longer U8.VCC
- net VCC_5V0: now also C13.1, C14.1, C7.1, C8.1, R19.2, R21.2, R22.2, TP_5V0.1, U11.OUT, U12.OUT, U8.VCC, USB_A.VCC, VR1.E; no longer J2.VBUS, JP1.VCC
Other:
- note added: "Assoc."
- note added: "Control Knob"
- note added: "LED Backlight Dimming for TFT"
- note added: "Power"
- note added: "RSSI"
- note added: "Radio On"
- note added: "Raspberry Pi 3 pin mappings: * GPIO2,3 = SDA1, SCL1 * GPIO14,15 = TXD0, RXD0 * GPIO20,21,22 = Encoder A, B, SW"
- note added: "Real-Time Clock"
- note added: "SD Active"
- note added: "TODO: * 5V hard wire points"
- note removed: "I²C Input from Raspberry Pi"
- note removed: "I²C LED Backlight Control for TFT"
- note removed: "Raspberry Pi 3 pin mappings: * GPIO2 = SDA1 * GPIO3 = SCL1 * GPIO14 = TXD0 * GPIO15 = RXD0"
- note removed: "TODO: * Add decoupling"
- note removed: "TODO: * Add decoupling * USB connections * Power status LEDs * XBee status LEDs * Add UI switches etc."
- moved on the sheet: C1, C2, C3, C4, C5, C6, D1, J1, J3, L1, L2, L3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
