File: hardware/SensorBoard/airball_sensor_board_v7.sch (EAGLE design)
At the start: 24 parts, among them J1 FEMALE 2x3

Commit message: Updated V7 board schematics
Connections:
- net VCC_3V3: now also MUX.#RESET
Changed lines of the file:
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@@
 <pinref part="U$2" gate="G$1" pin="VIN"/>
 <wire x1="175.26" y1="124.46" x2="180.34" y2="124.46" width="0.1524" layer="91"/>
+<pinref part="MUX" gate="G$1" pin="#RESET"/>
+<wire x1="40.64" y1="124.46" x2="38.1" y2="124.46" width="0.1524" layer="91"/>
+<wire x1="38.1" y1="124.46" x2="38.1" y2="160.02" width="0.1524" layer="91"/>
 </segment>
 </net>
